File: AR488-common/AR488-ESP32.sch (KiCad schematic (older format))
At the start: 9 parts, among them J1 Conn_02x12_Top_Bottom, J2 Conn_02x12_Odd_Even, J3 Barrel_Jack, J4 Screw_Terminal_01x02, U2 SN75162BDW, U3 SN75160BDW

Commit message: Better pin assignment for the inter-PCB connector
Parts:
- J1: value Conn_02x12_Top_Bottom -> GPIB-24
- renumbered U3 to U1
Connections:
- net +5V: now also J2.10 (Pin_10), J2.9 (Pin_9); no longer J2.21 (Pin_21), J2.22 (Pin_22)
- net ATN_a: now also J2.20 (Pin_20); no longer J2.14 (Pin_14)
- net D2: now also J2.2 (Pin_2); no longer J2.3 (Pin_3)
- net D3: now also J2.3 (Pin_3); no longer J2.5 (Pin_5)
- net D4: now also J2.4 (Pin_4); no longer J2.7 (Pin_7)
- net D5: now also J2.5 (Pin_5); no longer J2.9 (Pin_9)
- net D6: now also J2.6 (Pin_6); no longer J2.11 (Pin_11)
- net D7: now also J2.7 (Pin_7); no longer J2.13 (Pin_13)
- net D8: now also J2.8 (Pin_8); no longer J2.15 (Pin_15)
- net DAV_a: now also J2.18 (Pin_18); no longer J2.10 (Pin_10)
- net DC: now also J2.24 (Pin_24); no longer J2.20 (Pin_20)
- net EOI_a: now also J2.17 (Pin_17); no longer J2.12 (Pin_12)
- net GND: now also J2.11 (Pin_11), J2.12 (Pin_12); no longer J2.19 (Pin_19), J2.24 (Pin_24)
- net IFC_a: now also J2.13 (Pin_13); no longer J2.4 (Pin_4)
- net NDAC_a: now also J2.16 (Pin_16); no longer J2.6 (Pin_6)
- net NRFD_a: now also J2.15 (Pin_15); no longer J2.8 (Pin_8)
- net REN_a: now also J2.14 (Pin_14); no longer J2.2 (Pin_2)
- net SC: now also J2.21 (Pin_21); no longer J2.18 (Pin_18)
- net SRQ_a: now also J2.19 (Pin_19); no longer J2.16 (Pin_16)
- net TE: now also J2.22 (Pin_22); no longer J2.17 (Pin_17)
Changed lines of the file:
@@
 $EndDescr
 $Comp
-L Interface:SN75160BDW U3
+L Interface:SN75160BDW U1
 U 1 1 6167419F
 P 5650 1800
-F 0 "U3" H 5650 2681 50  0000 C CNN
-F 1 "SN75160BDW" H 5650 2590 50  0000 C CNN
+F 0 "U1" H 5900 2475 50  0000 C CNN
+F 1 "SN75160BDW" H 6025 1100 50  0000 C CNN
 F 2 "Package_SO:SOIC-20W_7.5x12.8mm_P1.27mm" H 5650 1500 50  0001 C CNN
 F 3 "http://www.ti.com/lit/ds/symlink/sn75160b.pdf" H 5600 2150 50  0001 C CNN
@@
 P 8100 2350
 F 0 "J1" H 8150 3067 50  0000 C CNN
-F 1 "Conn_02x12_Top_Bottom" H 8150 2976 50  0000 C CNN
+F 1 "GPIB-24" H 8150 2976 50  0000 C CNN
 F 2 "misc:CENTRONICS-24" H 8100 2350 50  0001 C CNN
 F 3 "~" H 8100 2350 50  0001 C CNN
@@
 P 5625 2950
 F 0 "#PWR04" H 5625 2800 50  0001 C CNN
-F 1 "+5V" H 5640 3123 50  0000 C CNN
+F 1 "+5V" H 5500 3025 50  0000 C CNN
 F 2 "" H 5625 2950 50  0001 C CNN
 F 3 "" H 5625 2950 50  0001 C CNN
@@
 U 1 1 617ED5E6
 P 3675 2175
-F 0 "J2" H 3725 2892 50  0000 C CNN
-F 1 "Conn_02x12_Odd_Even" H 3725 2801 50  0000 C CNN
+F 0 "J2" H 3725 2800 50  0000 C CNN
+F 1 "Conn_02x12_Odd_Even" H 3725 2801 50  0001 C CNN
 F 2 "Connector_PinSocket_2.54mm:PinSocket_2x12_P2.54mm_Vertical" H 3675 2175 50  0001 C CNN
 F 3 "~" H 3675 2175 50  0001 C CNN
@@
 Text GLabel 3475 1675 0    50   Input ~ 0
 D1
+Text GLabel 3975 1675 2    50   Input ~ 0
+D2
 Text GLabel 3475 1775 0    50   Input ~ 0
-D2
+D3
+Text GLabel 3975 1775 2    50   Input ~ 0
+D4
 Text GLabel 3475 1875 0    50   Input ~ 0
-D3
+D5
+Text GLabel 3975 1875 2    50   Input ~ 0
+D6
 Text GLabel 3475 1975 0    50   Input ~ 0
-D4
-Text GLabel 3475 2075 0    50   Input ~ 0
-D5
-Text GLabel 3475 2175 0    50   Input ~ 0
-D6
+D7
+Text GLabel 3975 1975 2    50   Input ~ 0
+D8
+Text GLabel 3975 2275 2    50   Input ~ 0
+REN_a
 Text GLabel 3475 2275 0    50   Input ~ 0
-D7
+IFC_a
+Text GLabel 3975 2375 2    50   Input ~ 0
+NDAC_a
 Text GLabel 3475 2375 0    50   Input ~ 0
-D8
-Text GLabel 3975 1675 2    50   Input ~ 0
-REN_a
-Text GLabel 3975 1775 2    50   Input ~ 0
-IFC_a
-Text GLabel 3975 1875 2    50   Input ~ 0
-NDAC_a
-Text GLabel 3975 1975 2    50   Input ~ 0
 NRFD_a
-Text GLabel 3975 2075 2    50   Input ~ 0
+Text GLabel 3975 2475 2    50   Input ~ 0
 DAV_a
-Text GLabel 3975 2175 2    50   Input ~ 0
+Text GLabel 3475 2475 0    50   Input ~ 0
 EOI_a
-Text GLabel 3975 2275 2    50   Input ~ 0
+Text GLabel 3975 2575 2    50   Input ~ 0
 ATN_a
-Text GLabel 3975 2375 2    50   Input ~ 0
+Text GLabel 3475 2575 0    50   Input ~ 0
 SRQ_a
-Text GLabel 3475 2475 0    50   Input ~ 0
+Text GLabel 3975 2675 2    50   Input ~ 0
 TE
-Text GLabel 3975 2475 2    50   Input ~ 0
+Text GLabel 3475 2675 0    50   Input ~ 0
 SC
-Text GLabel 3975 2575 2    50   Input ~ 0
+Text GLabel 3975 2775 2    50   Input ~ 0
 DC
 $Comp
 L power:GND #PWR010
 U 1 1 6180B39E
-P 3975 2775
-F 0 "#PWR010" H 3975 2525 50  0001 C CNN
-F 1 "GND" H 3980 2602 50  0000 C CNN
-F 2 "" H 3975 2775 50  0001 C CNN
-F 3 "" H 3975 2775 50  0001 C CNN
-	1    3975 2775
-	1    0    0    -1
+P 3975 2175
+F 0 "#PWR010" H 3975 1925 50  0001 C CNN
+F 1 "GND" V 3980 2002 50  0000 C CNN
+F 2 "" H 3975 2175 50  0001 C CNN
+F 3 "" H 3975 2175 50  0001 C CNN
+	1    3975 2175
+	0    -1   -1   0
 $EndComp
 $Comp
 L power:GND #PWR03
 U 1 1 6180BA39
+P 3475 2175
+F 0 "#PWR03" H 3475 1925 50  0001 C CNN
+F 1 "GND" V 3480 2002 50  0000 C CNN
+F 2 "" H 3475 2175 50  0001 C CNN
+F 3 "" H 3475 2175 50  0001 C CNN
+	1    3475 2175
+	0    1    1    0
+$EndComp
+$Comp
+L power:+5V #PWR09
+U 1 1 6180BF0B
+P 3975 2075
+F 0 "#PWR09" H 3975 1925 50  0001 C CNN
+F 1 "+5V" V 3975 2275 50  0000 C CNN
+F 2 "" H 3975 2075 50  0001 C CNN
+F 3 "" H 3975 2075 50  0001 C CNN
+	1    3975 2075
+	0    1    1    0
+$EndComp
+$Comp
+L power:+5V #PWR02
+U 1 1 6180CB7D
+P 3475 2075
+F 0 "#PWR02" H 3475 1925 50  0001 C CNN
+F 1 "+5V" V 3475 2275 50  0000 C CNN
+F 2 "" H 3475 2075 50  0001 C CNN
+F 3 "" H 3475 2075 50  0001 C CNN
+	1    3475 2075
+	0    -1   -1   0
+$EndComp
+$Comp
+L power:GND #PWR01
+U 1 1 6180D3A4
 P 3475 2775
-F 0 "#PWR03" H 3475 2525 50  0001 C CNN
-F 1 "GND" H 3480 2602 50  0000 C CNN
+F 0 "#PWR01" H 3475 2525 50  0001 C CNN
+F 1 "GND" V 3475 2575 50  0000 C CNN
 F 2 "" H 3475 2775 50  0001 C CNN
 F 3 "" H 3475 2775 50  0001 C CNN
 	1    3475 2775
-	1    0    0    -1
-$EndComp
-$Comp
-L power:+5V #PWR09
-U 1 1 6180BF0B
-P 3975 2675
-F 0 "#PWR09" H 3975 2525 50  0001 C CNN
-F 1 "+5V" H 3990 2848 50  0000 C CNN
-F 2 "" H 3975 2675 50  0001 C CNN
-F 3 "" H 3975 2675 50  0001 C CNN
-	1    3975 2675
-	0    1    1    0
-$EndComp
-$Comp
-L power:+5V #PWR02
-U 1 1 6180CB7D
-P 3475 2675
-F 0 "#PWR02" H 3475 2525 50  0001 C CNN
-F 1 "+5V" H 3490 2848 50  0000 C CNN
-F 2 "" H 3475 2675 50  0001 C CNN
-F 3 "" H 3475 2675 50  0001 C CNN
-	1    3475 2675
-	0    -1   -1   0
-$EndComp
-$Comp
-L power:GND #PWR01
-U 1 1 6180D3A4
-P 3475 2575
-F 0 "#PWR01" H 3475 2325 50  0001 C CNN
-F 1 "GND" H 3480 2402 50  0000 C CNN
-F 2 "" H 3475 2575 50  0001 C CNN
-F 3 "" H 3475 2575 50  0001 C CNN
-	1    3475 2575
 	0    1    1    0
 $EndComp
@@
 U 1 1 6180EAFE
 P 3675 3575
-F 0 "C1" H 3766 3621 50  0000 L CNN
-F 1 "10u" H 3766 3530 50  0000 L CNN
+F 0 "C1" H 3500 3650 50  0000 L CNN
+F 1 "10u" H 3450 3550 50  0000 L CNN
 F 2 "Capacitor_Tantalum_SMD:CP_EIA-7132-20_AVX-U" H 3675 3575 50  0001 C CNN
 F 3 "~" H 3675 3575 50  0001 C CNN
@@
 U 1 1 618102D7
 P 3900 3575
-F 0 "C2" H 3992 3621 50  0000 L CNN
-F 1 "100n" H 3992 3530 50  0000 L CNN
+F 0 "C2" H 3800 3650 50  0000 L CNN
+F 1 "100n" H 3900 3500 50  0000 L CNN
 F 2 "Capacitor_SMD:C_1206_3216Metric" H 3900 3575 50  0001 C CNN
 F 3 "~" H 3900 3575 50  0001 C CNN
@@
 U 1 1 618111BF
 P 4150 3575
-F 0 "C3" H 4242 3621 50  0000 L CNN
-F 1 "100n" H 4242 3530 50  0000 L CNN
+F 0 "C3" H 4025 3650 50  0000 L CNN
+F 1 "100n" H 4150 3500 50  0000 L CNN
 F 2 "Capacitor_SMD:C_1206_3216Metric" H 4150 3575 50  0001 C CNN
 F 3 "~" H 4150 3575 50  0001 C CNN
@@
 U 1 1 6182B7AF
 P 3025 3600
-F 0 "J3" H 3082 3917 50  0000 C CNN
-F 1 "Barrel_Jack" H 3082 3826 50  0000 C CNN
+F 0 "J3" H 2975 3800 50  0000 C CNN
+F 1 "Barrel_Jack" H 3082 3826 50  0001 C CNN
 F 2 "Connector_BarrelJack:BarrelJack_CUI_PJ-063AH_Horizontal" H 3075 3560 50  0001 C CNN
 F 3 "~" H 3075 3560 50  0001 C CNN
@@
 U 1 1 618381F0
 P 2975 4250
-F 0 "J4" H 2893 3925 50  0000 C CNN
-F 1 "Screw_Terminal_01x02" H 2893 4016 50  0000 C CNN
+F 0 "J4" H 2975 4050 50  0000 C CNN
+F 1 "Screw_Terminal_01x02" H 2250 4175 50  0001 C CNN
 F 2 "TerminalBlock:TerminalBlock_Altech_AK300-2_P5.00mm" H 2975 4250 50  0001 C CNN
 F 3 "~" H 2975 4250 50  0001 C CNN
@@
 $EndComp
 $Comp
-L power:GND #PWR?
+L power:GND #PWR0104
 U 1 1 6184381A
 P 3250 4300
-F 0 "#PWR?" H 3250 4050 50  0001 C CNN
+F 0 "#PWR0104" H 3250 4050 50  0001 C CNN
 F 1 "GND" H 3255 4127 50  0000 C CNN
 F 2 "" H 3250 4300 50  0001 C CNN
@@
 $EndComp
 $Comp
-L power:+5V #PWR?
+L power:+5V #PWR0105
 U 1 1 61843BAE
 P 3250 4125
-F 0 "#PWR?" H 3250 3975 50  0001 C CNN
+F 0 "#PWR0105" H 3250 3975 50  0001 C CNN
 F 1 "+5V" H 3265 4298 50  0000 C CNN
 F 2 "" H 3250 4125 50  0001 C CNN
@@
 U 1 1 6167818E
 P 5625 3650
-F 0 "U2" H 5625 4531 50  0000 C CNN
-F 1 "SN75162BDW" H 5625 4440 50  0000 C CNN
+F 0 "U2" H 5875 4325 50  0000 C CNN
+F 1 "SN75162BDW" H 5975 2925 50  0000 C CNN
 F 2 "Package_SO:SOIC-24W_7.5x15.4mm_P1.27mm" H 5625 3370 50  0001 C CNN
 F 3 "http://www.ti.com/lit/ds/symlink/sn75162b.pdf" H 5575 4000 50  0001 C CNN
@@
 $EndComp
 $Comp
-L power:GND #PWR?
+L power:GND #PWR0106
 U 1 1 6180BA51
 P 6025 4000
-F 0 "#PWR?" H 6025 3750 50  0001 C CNN
-F 1 "GND" H 6030 3827 50  0000 C CNN
+F 0 "#PWR0106" H 6025 3750 50  0001 C CNN
+F 1 "GND" V 6025 3800 50  0000 C CNN
 F 2 "" H 6025 4000 50  0001 C CNN
 F 3 "" H 6025 4000 50  0001 C CNN
@@
 DC
 $Comp
-L power:+5V #PWR?
+L power:+5V #PWR0107
 U 1 1 6180C427
 P 6025 4200
-F 0 "#PWR?" H 6025 4050 50  0001 C CNN
-F 1 "+5V" H 6040 4373 50  0000 C CNN
+F 0 "#PWR0107" H 6025 4050 50  0001 C CNN
+F 1 "+5V" V 6025 4400 50  0000 C CNN
 F 2 "" H 6025 4200 50  0001 C CNN
 F 3 "" H 6025 4200 50  0001 C CNN
