File: AR488-arduino-nano/AR488-arduino-nano.kicad_pcb (KiCad board)
At the start: 2 copper layers, 63.5 x 50 mm, 7 parts, among them J2 Conn_02x12_Odd_Even

Commit message: Several minor fixes and adjustments in PCBs
Parts:
- moved REF** 6.62 mm to (119.5, 97.0)
- moved REF** 0.15 mm to (71.4, 108.2)
- moved REF** 0.13 mm to (118.2, 108.2)
